Commit message: wip: urdf update for u18

File: gym_gazebo/envs/assets/urdf/kobuki_urdf/urdf/kobuki_gazebo.urdf.xacro (robot description, xacro)
@@ -9,4 +9,12 @@
 	    <minDepth>0.001</minDepth>
 	    <maxVel>1.0</maxVel>
+      <sensor type="contact" name="wheel_drop_left">
+        <always_on>1</always_on>
+        <update_rate>50.0</update_rate>
+        <visualize>true</visualize>
+        <contact>
+          <collision>wheel_left_link_collision</collision>
+        </contact>
+      </sensor>
 	  </gazebo>
 	  <gazebo reference="wheel_right_link">
@@ -17,4 +25,12 @@
 	    <minDepth>0.001</minDepth>
 	    <maxVel>1.0</maxVel>
+      <sensor type="contact" name="wheel_drop_right">
+        <always_on>1</always_on>
+        <update_rate>50.0</update_rate>
+        <visualize>true</visualize>
+        <contact>
+          <collision>wheel_right_link_collision</collision>
+        </contact>
+      </sensor>
 	  </gazebo>
 	  <gazebo reference="caster_front_link">
@@ -175,4 +191,6 @@
 	      <bumper_name>bumpers</bumper_name>
         <imu_name>imu</imu_name>
+        <wheel_drop_left_sensor_name>wheel_drop_left</wheel_drop_left_sensor_name>
+        <wheel_drop_right_sensor_name>wheel_drop_right</wheel_drop_right_sensor_name>
 	    </plugin>
 	  </gazebo>
